File: njordr-board/njordr-board.kicad_sch (KiCad schematic)
At the start: 3 parts, among them J1 Conn_01x06, J2 Conn_01x06, J3 Conn_01x06

Commit message: board: Improve board markings
- rotate reference labels
- add connector description
- add logo
Parts:
- J1: Label (none) -> ECH; Label2 (none) -> GND; Label3 (none) -> 3V3; Label4 (none) -> RXE; Label5 (none) -> INH; Label6 (none) -> INL
- J2: Label (none) -> EDG
- J3: Label (none) -> ENV
Changed lines of the file:
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@@
+			)
+		)
+		(property "Label" "EDG"
+			(at 60.96 91.44 0)
+			(effects
+				(font
+					(size 1.27 1.27)
+				)
+				(hide yes)
 			)
 		)
@@
 			)
 		)
+		(property "Label" "ENV"
+			(at 60.96 116.84 0)
+			(effects
+				(font
+					(size 1.27 1.27)
+				)
+				(hide yes)
+			)
+		)
 		(pin "6"
 		)
@@
 			(at 60.96 66.04 0)
 			(effects
+				(font
+					(size 1.27 1.27)
+				)
+				(hide yes)
+			)
+		)
+		(property "Label" "ECH"
+			(at 60.96 66.04 0)
+			(effects
+				(font
+					(size 1.27 1.27)
+				)
+				(hide yes)
+			)
+		)
+		(property "Label2" "GND"
+			(at 60.96 66.04 0)
+			(effects
+				(font
+					(size 1.27 1.27)
+				)
+				(hide yes)
+			)
+		)
+		(property "Label3" "3V3"
+			(at 60.96 66.04 0)
+			(effects
+				(font
+					(size 1.27 1.27)
+				)
+				(hide yes)
+			)
+		)
+		(property "Label4" "RXE"
+			(at 60.96 66.04 0)
+			(effects
+				(font
+					(size 1.27 1.27)
+				)
+				(hide yes)
+			)
+		)
+		(property "Label5" "INH"
+			(at 60.96 66.04 0)
+			(effects
+				(font
+					(size 1.27 1.27)
+				)
+				(hide yes)
+			)
+		)
+		(property "Label6" "INL"
+			(at 60.96 66.04 0)
+			(effects

Commit message: njordr-board: Use updated library symbols and packages
Parts:
- J1, J2, J3: footprint njordr:PinHeader_1x06_P2.54mm_Vertical -> njordr:PinHeader-1x06-P2.54mm-Vertical
Changed lines of the file:
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@@
 			)
 		)
-		(property "Footprint" "njordr:PinHeader_1x06_P2.54mm_Vertical"
+		(property "Footprint" "njordr:PinHeader-1x06-P2.54mm-Vertical"
 			(at 60.96 91.44 0)
 			(effects
@@
 			)
 		)
-		(property "Footprint" "njordr:PinHeader_1x06_P2.54mm_Vertical"
+		(property "Footprint" "njordr:PinHeader-1x06-P2.54mm-Vertical"
 			(at 60.96 116.84 0)
 			(effects
@@
 			)
 		)
-		(property "Footprint" "njordr:PinHeader_1x06_P2.54mm_Vertical"
+		(property "Footprint" "njordr:PinHeader-1x06-P2.54mm-Vertical"
 			(at 60.96 66.04 0)
 			(effects
