File: njordr-board/sonic-channel.kicad_sch (KiCad schematic)
At the start: 26 parts, among them Q101 2N7002, Q102 2N7002, T101 TestPoint, T102 TestPoint, T103 TestPoint, T104 TestPoint, T105 TestPoint, T106 TestPoint, T107 TestPoint

Commit message: board: Improve board markings
- rotate reference labels
- add connector description
- add logo
Parts:
- T101: Label (none) -> RAW
- T106: Label (none) -> SH
- T107: Label (none) -> SL
Changed lines of the file:
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@@
+			)
+		)
+		(property "Label" "SL"
+			(at 154.94 105.41 0)
+			(effects
+				(font
+					(size 1.27 1.27)
+				)
+				(hide yes)
 			)
 		)
@@
 			)
 		)
+		(property "Label" "SH"
+			(at 163.83 105.41 0)
+			(effects
+				(font
+					(size 1.27 1.27)
+				)
+				(hide yes)
+			)
+		)
 		(pin "1"
 		)
@@
 			(at 260.35 66.04 0)
 			(effects
+				(font
+					(size 1.27 1.27)
+				)
+				(hide yes)
+			)
+		)
+		(property "Label" "RAW"
+			(at 260.35 66.04 0)
+			(effects

Commit message: njordr-board: Use updated library symbols and packages
Parts:
- C101, C102, C105, C106, C107, C108: footprint njordr:C_0603_1608Metric_Pad1.08x0.95mm_HandSolder -> njordr:C-0603-HandSolder
- C103: footprint njordr:C_1206_3216Metric_Pad1.33x1.80mm_HandSolder -> njordr:C-1206-HandSolder
- C104: footprint njordr:C_0805_2012Metric_Pad1.18x1.45mm_HandSolder -> njordr:C-0805-HandSolder
- D101, D102: footprint njordr:D_SOD-323_HandSoldering -> njordr:D-SOD-323-HandSolder
- L101: footprint njordr:L_Axial_L12.0mm_D5.0mm_P15.24mm_Horizontal_Fastron_MISC -> njordr:L-Axial-L12.0-D5.0-P15.24
- R101, R102, R103, R104: footprint njordr:R_0603_1608Metric_Pad0.98x0.95mm_HandSolder -> njordr:R-0603-HandSolder
- R105: footprint njordr:R_0805_2012Metric_Pad1.20x1.40mm_HandSolder -> njordr:R-0805-HandSolder
- ST101: footprint njordr:Buzzer_D14mm_H9mm_P5mm -> njordr:CUSA-TR65-065-2200-TH68
- T101, T102, T103, T104, T105, T106, T107: footprint njordr:TestPoint_Pad_1.0x1.0mm -> njordr:TestPoint-Pad-1.0x1.0
Changed lines of the file:
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@@
 			)
 		)
-		(property "Footprint" "njordr:R_0603_1608Metric_Pad0.98x0.95mm_HandSolder"
+		(property "Footprint" "njordr:R-0603-HandSolder"
 			(at 74.93 86.868 90)
 			(effects
@@
 			)
 		)
-		(property "Datasheet" "https://jlcpcb.com/partdetail/23586-0603WAF100JT5E/C22859"
+		(property "Datasheet" "~"
 			(at 74.93 85.09 0)
 			(effects
@@
 			)
 		)
-		(property "Footprint" "njordr:C_0805_2012Metric_Pad1.18x1.45mm_HandSolder"
+		(property "Footprint" "njordr:C-0805-HandSolder"
 			(at 261.3152 128.27 0)
 			(effects
@@
 			)
 		)
-		(property "Datasheet" "https://jlcpcb.com/partdetail/46786-CL21A226MAQNNNE/C45783"
+		(property "Datasheet" "~"
 			(at 260.35 124.46 0)
 			(effects
@@
 			)
 		)
-		(property "Footprint" "njordr:TestPoint_Pad_1.0x1.0mm"
+		(property "Footprint" "njordr:TestPoint-Pad-1.0x1.0"
 			(at 160.02 105.41 0)
 			(effects
@@
 			)
 		)
-		(property "Footprint" "njordr:TestPoint_Pad_1.0x1.0mm"
+		(property "Footprint" "njordr:TestPoint-Pad-1.0x1.0"
 			(at 57.15 82.55 0)
 			(effects
@@
 			)
 		)
-		(property "Footprint" "njordr:L_Axial_L12.0mm_D5.0mm_P15.24mm_Horizontal_Fastron_MISC"
+		(property "Footprint" "njordr:L-Axial-L12.0-D5.0-P15.24"
 			(at 97.79 109.22 0)
 			(effects
@@
 			)
 		)
-		(property "Datasheet" "https://cz.mouser.com/ProductDetail/70-IRF46ER822K"
+		(property "Datasheet" "~"
 			(at 97.79 109.22 0)
 			(effects
@@
 			)
 		)
-		(property "Footprint" "njordr:C_0603_1608Metric_Pad1.08x0.95mm_HandSolder"
+		(property "Footprint" "njordr:C-0603-HandSolder"
 			(at 246.6848 80.01 0)
 			(effects
@@
 			)
 		)
-		(property "Datasheet" "https://jlcpcb.com/partdetail/2016-CL10C331JB8NNNC/C1664"
+		(property "Datasheet" "~"
 			(at 247.65 76.2 0)
 			(effects
@@
 			)
 		)
-		(property "Datasheet" "https://jlcpcb.com/partdetail/9040-2N7002/C8545"
+		(property "Datasheet" "https://www.onsemi.com/pub/Collateral/NDS7002A-D.PDF"
 			(at 92.71 88.9 0)
 			(effects
@@
 			)
 		)
-		(property "Footprint" "njordr:C_0603_1608Metric_Pad1.08x0.95mm_HandSolder"
+		(property "Footprint" "njordr:C-0603-HandSolder"
 			(at 235.9152 128.27 0)
 			(effects
@@
 			)
 		)
-		(property "Datasheet" "https://jlcpcb.com/api/file/downloadByFileSystemAccessId/8579707083955945472"
+		(property "Datasheet" "~"
 			(at 234.95 124.46 0)
 			(effects
@@
 			)
 		)
-		(property "Footprint" "njordr:C_1206_3216Metric_Pad1.33x1.80mm_HandSolder"
+		(property "Footprint" "njordr:C-1206-HandSolder"
 			(at 250.19 67.6148 0)
 			(effects
@@
 			)
 		)
-		(property "Datasheet" "https://jlcpcb.com/partdetail/9721-1206B102K202NT/C9196"
+		(property "Datasheet" "~"
 			(at 254 68.58 0)
 			(effects
@@
 			)
 		)
-		(property "Description" "Ceramic 1n 1206 2kV"
+		(property "Description" "Unpolarized capacitor"
 			(at 254 68.58 0)
 			(effects
@@
 			)
 		)
-		(property "Footprint" "njordr:R_0603_1608Metric_Pad0.98x0.95mm_HandSolder"
+		(property "Footprint" "njordr:R-0603-HandSolder"
 			(at 74.93 122.428 90)
 			(effects
@@
 			)
 		)
-		(property "Datasheet" "https://jlcpcb.com/partdetail/23586-0603WAF100JT5E/C22859"
+		(property "Datasheet" "~"
 			(at 74.93 120.65 0)
 			(effects
@@
 			)
 		)
-		(property "Footprint" "njordr:TestPoint_Pad_1.0x1.0mm"
+		(property "Footprint" "njordr:TestPoint-Pad-1.0x1.0"
 			(at 57.15 118.11 0)
 			(effects
@@
 			)
 		)
-		(property "Footprint" "njordr:R_0603_1608Metric_Pad0.98x0.95mm_HandSolder"
+		(property "Footprint" "njordr:R-0603-HandSolder"
 			(at 153.162 119.38 90)
 			(effects
@@
 			)
 		)
-		(property "Datasheet" "https://jlcpcb.com/partdetail/23586-0603WAF100JT5E/C22859"
+		(property "Datasheet" "~"
 			(at 154.94 119.38 0)
 			(effects
@@
 			)
 		)
-		(property "Footprint" "njordr:TestPoint_Pad_1.0x1.0mm"
+		(property "Footprint" "njordr:TestPoint-Pad-1.0x1.0"
 			(at 168.91 105.41 0)
 			(effects
@@
 			)
 		)
-		(property "Footprint" "njordr:Buzzer_D14mm_H9mm_P5mm"
+		(property "Footprint" "njordr:CUSA-TR65-065-2200-TH68"
 			(at 173.101 110.49 0)
 			(effects
@@
 			)
 		)
-		(property "Datasheet" "https://jlcpcb.com/partdetail/9040-2N7002/C8545"
+		(property "Datasheet" "https://www.onsemi.com/pub/Collateral/NDS7002A-D.PDF"
 			(at 92.71 124.46 0)
 			(effects
@@
 			)
 		)
-		(property "Footprint" "njordr:D_SOD-323_HandSoldering"
+		(property "Footprint" "njordr:D-SOD-323-HandSolder"
 			(at 241.935 76.2 0)
 			(effects
@@
 			)
 		)
-		(property "Datasheet" "https://jlcpcb.com/partdetail/2485-1N4148WS/C2128"
+		(property "Datasheet" "https://www.vishay.com/docs/85751/1n4148ws.pdf"
 			(at 237.49 76.2 0)
 			(effects
@@
 			)
 		)
-		(property "Footprint" "njordr:C_0603_1608Metric_Pad1.08x0.95mm_HandSolder"
+		(property "Footprint" "njordr:C-0603-HandSolder"
 			(at 78.74 96.8248 0)
 			(effects
@@
 			)
 		)
-		(property "Datasheet" "https://jlcpcb.com/api/file/downloadByFileSystemAccessId/8579707083955945472"
+		(property "Datasheet" "~"
 			(at 74.93 97.79 0)
 			(effects
@@
 			)
 		)
-		(property "Footprint" "njordr:TestPoint_Pad_1.0x1.0mm"
+		(property "Footprint" "njordr:TestPoint-Pad-1.0x1.0"
 			(at 57.15 95.25 0)
 			(effects
@@
 			)
 		)
-		(property "Footprint" "njordr:R_0805_2012Metric_Pad1.20x1.40mm_HandSolder"
+		(property "Footprint" "njordr:R-0805-HandSolder"
 			(at 222.25 70.358 90)
 			(effects
@@
 			)
 		)
-		(property "Datasheet" "https://jlcpcb.com/partdetail/23889-0603WAF4701T5E/C23162"
+		(property "Datasheet" "~"
 			(at 222.25 68.58 0)
 			(effects
@@
 			)
 		)
-		(property "Description" "0805 150V"
+		(property "Description" "Resistor"
 			(at 222.25 68.58 0)
 			(effects
@@
 			)
 		)
-		(property "Footprint" "njordr:TestPoint_Pad_1.0x1.0mm"
+		(property "Footprint" "njordr:TestPoint-Pad-1.0x1.0"
 			(at 265.43 66.04 0)
 			(effects
@@
 			)
 		)
-		(property "Footprint" "njordr:C_0603_1608Metric_Pad1.08x0.95mm_HandSolder"
+		(property "Footprint" "njordr:C-0603-HandSolder"
 			(at 213.0552 128.27 0)
 			(effects
@@
 			)
 		)
-		(property "Datasheet" "https://jlcpcb.com/api/file/downloadByFileSystemAccessId/8579707083955945472"
+		(property "Datasheet" "~"
 			(at 212.09 124.46 0)
 			(effects
@@
 			)
 		)
-		(property "Footprint" "njordr:C_0603_1608Metric_Pad1.08x0.95mm_HandSolder"
+		(property "Footprint" "njordr:C-0603-HandSolder"
 			(at 224.4852 128.27 0)
 			(effects
@@
 			)
 		)
-		(property "Datasheet" "https://jlcpcb.com/api/file/downloadByFileSystemAccessId/8579707083955945472"
+		(property "Datasheet" "~"
 			(at 223.52 124.46 0)
 			(effects
@@
 			)
 		)
-		(property "Footprint" "njordr:C_0603_1608Metric_Pad1.08x0.95mm_HandSolder"
+		(property "Footprint" "njordr:C-0603-HandSolder"
 			(at 248.6152 128.27 0)
 			(effects
@@
 			)
 		)
-		(property "Datasheet" "https://jlcpcb.com/api/file/downloadByFileSystemAccessId/8556213788459761664"
+		(property "Datasheet" "~"
 			(at 247.65 124.46 0)
 			(effects
@@
 			)
 		)
-		(property "Footprint" "njordr:R_0603_1608Metric_Pad0.98x0.95mm_HandSolder"
+		(property "Footprint" "njordr:R-0603-HandSolder"
 			(at 214.122 76.2 90)
 			(effects
@@
 			)
 		)
-		(property "Datasheet" "https://jlcpcb.com/partdetail/4597-0603WAF2201T5E/C4190"
+		(property "Datasheet" "~"
 			(at 215.9 76.2 0)
 			(effects
@@
 			)
 		)
-		(property "Footprint" "njordr:TestPoint_Pad_1.0x1.0mm"
+		(property "Footprint" "njordr:TestPoint-Pad-1.0x1.0"
 			(at 57.15 106.68 0)
 			(effects
@@
 			)
 		)
-		(property "Footprint" "njordr:D_SOD-323_HandSoldering"
+		(property "Footprint" "njordr:D-SOD-323-HandSolder"
 			(at 224.155 76.2 0)
 			(effects
@@
 			)
 		)
-		(property "Datasheet" "https://jlcpcb.com/partdetail/2485-1N4148WS/C2128"
+		(property "Datasheet" "https://www.vishay.com/docs/85751/1n4148ws.pdf"
 			(at 228.6 76.2 0)
 			(effects
