File: sensor-board/sensor-board.kicad_pcb (KiCad board)
At the start: 4 copper layers, 41.5 x 40 mm, 13 parts, among them J1 SM04B-SRSS-TB(LFSN), U1 HDC2010YPAR, U2 HP203B

Commit message: repo: Rename project from njordr to vetroplach
- vetroplach is a more playful name for the anemometer, suggested by
  the author's wife, replacing the Norse god name
- the board and firmware directories, the shared KiCad symbol and
  footprint libraries, the CI workflows, and every in-file reference
  change in one step so the tree never mixes the two names
Parts:
- C1, C2, C3, C5: footprint njordr:C-0603-HandSolder -> vetroplach:C-0603-HandSolder
- C4, C6: footprint njordr:C-0805-HandSolder -> vetroplach:C-0805-HandSolder
- J1: footprint njordr:SM04B-SRSS-TB -> vetroplach:SM04B-SRSS-TB
- R1, R2, R5, R6: footprint njordr:R-0603-HandSolder -> vetroplach:R-0603-HandSolder
- U1: footprint njordr:DSBGA-6-1.5x1.5 -> vetroplach:DSBGA-6-1.5x1.5
- U2: footprint njordr:QFN-8-HP203B -> vetroplach:QFN-8-HP203B
Changed lines of the file:
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@@
 	(net 12 "unconnected-(U1-DRDY_{slash}_INT-PadC2)")
 	(net 13 "Net-(U1-SDA)")
-	(footprint "njordr:DSBGA-6-1.5x1.5"
+	(footprint "vetroplach:DSBGA-6-1.5x1.5"
 		(layer "F.Cu")
 		(at 170.542716 81.305647 30)
@@
 		)
 	)
-	(footprint "njordr:C-0603-HandSolder"
+	(footprint "vetroplach:C-0603-HandSolder"
 		(layer "F.Cu")
 		(at 141.690283 78.751646 -30)
@@
 		)
 	)
-	(footprint "njordr:C-0805-HandSolder"
+	(footprint "vetroplach:C-0805-HandSolder"
 		(layer "F.Cu")
 		(at 148.750001 107.574998)
@@
 		)
 	)
-	(footprint "njordr:SM04B-SRSS-TB"
+	(footprint "vetroplach:SM04B-SRSS-TB"
 		(layer "F.Cu")
 		(at 155.35523 106.282955)
@@
 		)
 	)
-	(footprint "njordr:QFN-8-HP203B"
+	(footprint "vetroplach:QFN-8-HP203B"
 		(layer "F.Cu")
 		(at 140.190288 81.349726 -30)
@@
 		)
 	)
-	(footprint "njordr:R-0603-HandSolder"
+	(footprint "vetroplach:R-0603-HandSolder"
 		(layer "F.Cu")
 		(at 139.056311 85.313824 -120)
@@
 		)
 	)
-	(footprint "njordr:R-0603-HandSolder"
+	(footprint "vetroplach:R-0603-HandSolder"
 		(layer "F.Cu")
 		(at 171.218631 84.416149 -60)
@@
 		)
 	)
-	(footprint "njordr:R-0603-HandSolder"
+	(footprint "vetroplach:R-0603-HandSolder"
 		(layer "F.Cu")
 		(at 172.941962 83.461262 -60)
@@
 		)
 	)
-	(footprint "njordr:R-0603-HandSolder"
+	(footprint "vetroplach:R-0603-HandSolder"
 		(layer "F.Cu")
 		(at 137.42613 84.37264 -120)
@@
 		)
 	)
-	(footprint "njordr:C-0603-HandSolder"
+	(footprint "vetroplach:C-0603-HandSolder"
 		(layer "F.Cu")
 		(at 169.318163 79.184655 30)
@@
 		)
 	)
-	(footprint "njordr:C-0603-HandSolder"
+	(footprint "vetroplach:C-0603-HandSolder"
 		(layer "F.Cu")
 		(at 148.749997 104.046941)
@@
 		)
 	)
-	(footprint "njordr:C-0603-HandSolder"
+	(footprint "vetroplach:C-0603-HandSolder"
 		(layer "F.Cu")
 		(at 161.999998 104.046943 180)
@@
 		)
 	)
-	(footprint "njordr:C-0805-HandSolder"
+	(footprint "vetroplach:C-0805-HandSolder"
 		(layer "F.Cu")
 		(at 162 107.575 180)
