File: sensor-board/sensor-board.kicad_sch (KiCad schematic)
At the start: 13 parts, among them J1 SM04B-SRSS-TB, U1 HDC2010YPAR, U2 HP203B

Commit message: repo: Rename project from njordr to vetroplach
- vetroplach is a more playful name for the anemometer, suggested by
  the author's wife, replacing the Norse god name
- the board and firmware directories, the shared KiCad symbol and
  footprint libraries, the CI workflows, and every in-file reference
  change in one step so the tree never mixes the two names
Parts:
- C1, C2, C3, C5: footprint njordr:C-0603-HandSolder -> vetroplach:C-0603-HandSolder
- C4, C6: footprint njordr:C-0805-HandSolder -> vetroplach:C-0805-HandSolder
- J1: footprint njordr:SM04B-SRSS-TB -> vetroplach:SM04B-SRSS-TB; symbol njordr:SM04B-SRSS-TB -> vetroplach:SM04B-SRSS-TB
- R1, R2, R5, R6: footprint njordr:R-0603-HandSolder -> vetroplach:R-0603-HandSolder
- U1: footprint njordr:DSBGA-6-1.5x1.5 -> vetroplach:DSBGA-6-1.5x1.5; symbol njordr:HDC2010YPAR -> vetroplach:HDC2010YPAR
- U2: footprint njordr:QFN-8-HP203B -> vetroplach:QFN-8-HP203B; symbol njordr:HP203B -> vetroplach:HP203B
Changed lines of the file:
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@@
 			)
 		)
-		(property "Footprint" "njordr:C-0603-HandSolder"
+		(property "Footprint" "vetroplach:C-0603-HandSolder"
 			(at 49.2252 67.31 0)
 			(effects
@@
 	)
 	(symbol
-		(lib_id "njordr:HDC2010YPAR")
+		(lib_id "vetroplach:HDC2010YPAR")
 		(at 68.58 58.42 0)
 		(unit 1)
@@
 			)
 		)
-		(property "Footprint" "njordr:DSBGA-6-1.5x1.5"
+		(property "Footprint" "vetroplach:DSBGA-6-1.5x1.5"
 			(at 100.33 153.34 0)
 			(effects
@@
 			)
 		)
-		(property "Footprint" "njordr:C-0603-HandSolder"
+		(property "Footprint" "vetroplach:C-0603-HandSolder"
 			(at 82.2452 135.89 0)
 			(effects
@@
 			)
 		)
-		(property "Footprint" "njordr:R-0603-HandSolder"
+		(property "Footprint" "vetroplach:R-0603-HandSolder"
 			(at 237.49 67.818 90)
 			(effects
@@
 			)
 		)
-		(property "Footprint" "njordr:C-0805-HandSolder"
+		(property "Footprint" "vetroplach:C-0805-HandSolder"
 			(at 93.6752 135.89 0)
 			(effects
@@
 			)
 		)
-		(property "Footprint" "njordr:R-0603-HandSolder"
+		(property "Footprint" "vetroplach:R-0603-HandSolder"
 			(at 111.76 62.738 90)
 			(effects
@@
 			)
 		)
-		(property "Footprint" "njordr:C-0603-HandSolder"
+		(property "Footprint" "vetroplach:C-0603-HandSolder"
 			(at 174.9552 69.85 0)
 			(effects
@@
 			)
 		)
-		(property "Footprint" "njordr:R-0603-HandSolder"
+		(property "Footprint" "vetroplach:R-0603-HandSolder"
 			(at 111.76 65.278 90)
 			(effects
@@
 			)
 		)
-		(property "Footprint" "njordr:C-0805-HandSolder"
+		(property "Footprint" "vetroplach:C-0805-HandSolder"
 			(at 116.5352 135.89 0)
 			(effects
@@
 	)
 	(symbol
-		(lib_id "njordr:HP203B")
+		(lib_id "vetroplach:HP203B")
 		(at 212.09 66.04 0)
 		(unit 1)
@@
 			)
 		)
-		(property "Footprint" "njordr:QFN-8-HP203B"
+		(property "Footprint" "vetroplach:QFN-8-HP203B"
 			(at 212.09 77.47 0)
 			(effects
@@
 	)
 	(symbol
-		(lib_id "njordr:SM04B-SRSS-TB")
+		(lib_id "vetroplach:SM04B-SRSS-TB")
 		(at 58.42 128.27 0)
 		(unit 1)
@@
 			)
 		)
-		(property "Footprint" "njordr:SM04B-SRSS-TB"
+		(property "Footprint" "vetroplach:SM04B-SRSS-TB"
 			(at 58.42 128.27 0)
 			(effects
@@
 			)
 		)
-		(property "Footprint" "njordr:C-0603-HandSolder"
+		(property "Footprint" "vetroplach:C-0603-HandSolder"
 			(at 105.1052 135.89 0)
 			(effects
@@
 			)
 		)
-		(property "Footprint" "njordr:R-0603-HandSolder"
+		(property "Footprint" "vetroplach:R-0603-HandSolder"
 			(at 237.49 65.278 90)
 			(effects
