File: vetroplach-board/controller.kicad_sch (KiCad schematic)
At the start: 21 parts, among them Q1 MMBT2222A, SW1 RST, SW2 BOOT, U4 ESP32-S3, U5 GD25QxxxEY, Y1 40 MHz, Y2 32.768 kHz

Commit message: repo: Rename project from njordr to vetroplach
- vetroplach is a more playful name for the anemometer, suggested by
  the author's wife, replacing the Norse god name
- the board and firmware directories, the shared KiCad symbol and
  footprint libraries, the CI workflows, and every in-file reference
  change in one step so the tree never mixes the two names
Parts:
- C10, C14, C15, C16, C4, C5, C8: footprint njordr:C-0603-HandSolder -> vetroplach:C-0603-HandSolder
Other:
- title: NJORDR-BOARD -> VETROPLACH-BOARD
Changed lines of the file:
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@@
 	(paper "A4")
 	(title_block
-		(title "NJORDR-BOARD")
+		(title "VETROPLACH-BOARD")
 		(date "2025-08-24")
 		(rev "0.1")
@@
 		)
 		(instances
-			(project "njordr-board"
+			(project "vetroplach-board"
 				(path "/837a3018-1957-4824-b018-c0ef83e9cb67/27a9dd2e-a3b6-499f-b81b-edb2a809ca38"
 					(reference "R8")
@@
 			)
 		)
-		(property "Footprint" "njordr:C-0603-HandSolder"
+		(property "Footprint" "vetroplach:C-0603-HandSolder"
 			(at 57.15 90.4748 0)
 			(effects
@@
 		)
 		(instances
-			(project "njordr-board"
+			(project "vetroplach-board"
 				(path "/837a3018-1957-4824-b018-c0ef83e9cb67/27a9dd2e-a3b6-499f-b81b-edb2a809ca38"
 					(reference "C10")
@@
 			)
 		)
-		(property "Footprint" "njordr:C-0603-HandSolder"
+		(property "Footprint" "vetroplach:C-0603-HandSolder"
 			(at 75.2348 48.26 0)
 			(effects
@@
 		)
 		(instances
-			(project "njordr-board"
+			(project "vetroplach-board"
 				(path "/837a3018-1957-4824-b018-c0ef83e9cb67/27a9dd2e-a3b6-499f-b81b-edb2a809ca38"
 					(reference "C16")
@@
 		)
 		(instances
-			(project "njordr-board"
+			(project "vetroplach-board"
 				(path "/837a3018-1957-4824-b018-c0ef83e9cb67/27a9dd2e-a3b6-499f-b81b-edb2a809ca38"
 					(reference "R4")
@@
 		)
 		(instances
-			(project "njordr-board"
+			(project "vetroplach-board"
 				(path "/837a3018-1957-4824-b018-c0ef83e9cb67/27a9dd2e-a3b6-499f-b81b-edb2a809ca38"
 					(reference "#PWR017")
@@
 		)
 		(instances
-			(project "njordr-board"
+			(project "vetroplach-board"
 				(path "/837a3018-1957-4824-b018-c0ef83e9cb67/27a9dd2e-a3b6-499f-b81b-edb2a809ca38"
 					(reference "#PWR013")
@@
 		)
 		(instances
-			(project "njordr-board"
+			(project "vetroplach-board"
 				(path "/837a3018-1957-4824-b018-c0ef83e9cb67/27a9dd2e-a3b6-499f-b81b-edb2a809ca38"
 					(reference "Y2")
@@
 		)
 		(instances
-			(project "njordr-board"
+			(project "vetroplach-board"
 				(path "/837a3018-1957-4824-b018-c0ef83e9cb67/27a9dd2e-a3b6-499f-b81b-edb2a809ca38"
 					(reference "#PWR025")
@@
 		)
 		(instances
-			(project "njordr-board"
+			(project "vetroplach-board"
 				(path "/837a3018-1957-4824-b018-c0ef83e9cb67/27a9dd2e-a3b6-499f-b81b-edb2a809ca38"
 					(reference "#PWR019")
@@
 		)
 		(instances
-			(project "njordr-board"
+			(project "vetroplach-board"
 				(path "/837a3018-1957-4824-b018-c0ef83e9cb67/27a9dd2e-a3b6-499f-b81b-edb2a809ca38"
 					(reference "#PWR038")
@@
 		)
 		(instances
-			(project "njordr-board"
+			(project "vetroplach-board"
 				(path "/837a3018-1957-4824-b018-c0ef83e9cb67/27a9dd2e-a3b6-499f-b81b-edb2a809ca38"
 					(reference "D2")
@@
 			)
 		)
-		(property "Footprint" "njordr:C-0603-HandSolder"
+		(property "Footprint" "vetroplach:C-0603-HandSolder"
 			(at 57.15 128.5748 0)
 			(effects
@@
 		)
 		(instances
-			(project "njordr-board"
+			(project "vetroplach-board"
 				(path "/837a3018-1957-4824-b018-c0ef83e9cb67/27a9dd2e-a3b6-499f-b81b-edb2a809ca38"
 					(reference "C15")
@@
 		)
 		(instances
-			(project "njordr-board"
+			(project "vetroplach-board"
 				(path "/837a3018-1957-4824-b018-c0ef83e9cb67/27a9dd2e-a3b6-499f-b81b-edb2a809ca38"
 					(reference "R5")
@@
 		)
 		(instances
-			(project "njordr-board"
+			(project "vetroplach-board"
 				(path "/837a3018-1957-4824-b018-c0ef83e9cb67/27a9dd2e-a3b6-499f-b81b-edb2a809ca38"
 					(reference "#PWR024")
@@
 		)
 		(instances
-			(project "njordr-board"
+			(project "vetroplach-board"
 				(path "/837a3018-1957-4824-b018-c0ef83e9cb67/27a9dd2e-a3b6-499f-b81b-edb2a809ca38"
 					(reference "Y1")
@@
 		)
 		(instances
-			(project "njordr-board"
+			(project "vetroplach-board"
 				(path "/837a3018-1957-4824-b018-c0ef83e9cb67/27a9dd2e-a3b6-499f-b81b-edb2a809ca38"
 					(reference "#PWR016")
@@
 		)
 		(instances
-			(project "njordr-board"
+			(project "vetroplach-board"
 				(path "/837a3018-1957-4824-b018-c0ef83e9cb67/27a9dd2e-a3b6-499f-b81b-edb2a809ca38"
 					(reference "#PWR022")
@@
 			)
 		)
-		(property "Footprint" "njordr:C-0603-HandSolder"
+		(property "Footprint" "vetroplach:C-0603-HandSolder"
 			(at 38.4048 48.26 0)
 			(effects
@@
 		)
 		(instances
-			(project "njordr-board"
+			(project "vetroplach-board"
 				(path "/837a3018-1957-4824-b018-c0ef83e9cb67/27a9dd2e-a3b6-499f-b81b-edb2a809ca38"
 					(reference "C4")
@@
 		)
 		(instances
-			(project "njordr-board"
+			(project "vetroplach-board"
 				(path "/837a3018-1957-4824-b018-c0ef83e9cb67/27a9dd2e-a3b6-499f-b81b-edb2a809ca38"
 					(reference "#PWR018")
@@
 			)
 		)
-		(property "Footprint" "njordr:C-0603-HandSolder"
+		(property "Footprint" "vetroplach:C-0603-HandSolder"
 			(at 57.15 118.4148 0)
 			(effects
@@
 		)
 		(instances
-			(project "njordr-board"
+			(project "vetroplach-board"
 				(path "/837a3018-1957-4824-b018-c0ef83e9cb67/27a9dd2e-a3b6-499f-b81b-edb2a809ca38"
 					(reference "C14")
@@
 		)
 		(instances
-			(project "njordr-board"
+			(project "vetroplach-board"
 				(path "/837a3018-1957-4824-b018-c0ef83e9cb67/27a9dd2e-a3b6-499f-b81b-edb2a809ca38"
 					(reference "#PWR027")
@@
 		)
 		(instances
-			(project "njordr-board"
+			(project "vetroplach-board"
 				(path "/837a3018-1957-4824-b018-c0ef83e9cb67/27a9dd2e-a3b6-499f-b81b-edb2a809ca38"
 					(reference "#PWR020")
@@
 		)
 		(instances
-			(project "njordr-board"
+			(project "vetroplach-board"
 				(path "/837a3018-1957-4824-b018-c0ef83e9cb67/27a9dd2e-a3b6-499f-b81b-edb2a809ca38"
 					(reference "SW2")
@@
 		)
 		(instances
-			(project "njordr-board"
+			(project "vetroplach-board"
 				(path "/837a3018-1957-4824-b018-c0ef83e9cb67/27a9dd2e-a3b6-499f-b81b-edb2a809ca38"
 					(reference "R7")
@@
 			)
 		)
-		(property "Footprint" "njordr:C-0603-HandSolder"
+		(property "Footprint" "vetroplach:C-0603-HandSolder"
 			(at 57.15 80.3148 0)
 			(effects
@@
 		)
 		(instances
-			(project "njordr-board"
+			(project "vetroplach-board"
 				(path "/837a3018-1957-4824-b018-c0ef83e9cb67/27a9dd2e-a3b6-499f-b81b-edb2a809ca38"
 					(reference "C8")
@@
 		)
 		(instances
-			(project "njordr-board"
+			(project "vetroplach-board"
 				(path "/837a3018-1957-4824-b018-c0ef83e9cb67/27a9dd2e-a3b6-499f-b81b-edb2a809ca38"
 					(reference "#PWR015")
@@
 		)
 		(instances
-			(project "njordr-board"
+			(project "vetroplach-board"
 				(path "/837a3018-1957-4824-b018-c0ef83e9cb67/27a9dd2e-a3b6-499f-b81b-edb2a809ca38"
 					(reference "R9")
@@
 		)
 		(instances
-			(project "njordr-board"
+			(project "vetroplach-board"
 				(path "/837a3018-1957-4824-b018-c0ef83e9cb67/27a9dd2e-a3b6-499f-b81b-edb2a809ca38"
 					(reference "#PWR023")
@@
 		)
 		(instances
-			(project "njordr-board"
+			(project "vetroplach-board"
 				(path "/837a3018-1957-4824-b018-c0ef83e9cb67/27a9dd2e-a3b6-499f-b81b-edb2a809ca38"
 					(reference "#PWR014")
@@
 		)
 		(instances
-			(project "njordr-board"
+			(project "vetroplach-board"
 				(path "/837a3018-1957-4824-b018-c0ef83e9cb67/27a9dd2e-a3b6-499f-b81b-edb2a809ca38"
 					(reference "#PWR021")
@@
 			)
 		)
-		(property "Footprint" "njordr:C-0603-HandSolder"
+		(property "Footprint" "vetroplach:C-0603-HandSolder"
 			(at 51.1048 48.26 0)
 			(effects
@@
 		)
 		(instances
-			(project "njordr-board"
+			(project "vetroplach-board"
 				(path "/837a3018-1957-4824-b018-c0ef83e9cb67/27a9dd2e-a3b6-499f-b81b-edb2a809ca38"
 					(reference "C5")
@@
 		)
 		(instances
-			(project "njordr-board"
+			(project "vetroplach-board"
 				(path "/837a3018-1957-4824-b018-c0ef83e9cb67/27a9dd2e-a3b6-499f-b81b-edb2a809ca38"
 					(reference "#PWR012")
@@
 		)
 		(instances
-			(project "njordr-board"
+			(project "vetroplach-board"
 				(path "/837a3018-1957-4824-b018-c0ef83e9cb67/27a9dd2e-a3b6-499f-b81b-edb2a809ca38"
 					(reference "Q1")
@@
 		)
 		(instances
-			(project "njordr-board"
+			(project "vetroplach-board"
 				(path "/837a3018-1957-4824-b018-c0ef83e9cb67/27a9dd2e-a3b6-499f-b81b-edb2a809ca38"
 					(reference "R6")
@@
 		)
 		(instances
-			(project "njordr-board"
+			(project "vetroplach-board"
 				(path "/837a3018-1957-4824-b018-c0ef83e9cb67/27a9dd2e-a3b6-499f-b81b-edb2a809ca38"
 					(reference "SW1")
