File: vetroplach-board/interface.kicad_sch (KiCad schematic)
At the start: 22 parts, among them IC1 DRV8300DPWR, J301 Conn_01x04, T3 TestPoint, T4 TestPoint, T5 TestPoint, T6 TestPoint, T8 TestPoint, U1 ESDU5V0H4, U2 MT3608, U6 AMS1117-3.3

Commit message: repo: Rename project from njordr to vetroplach
- vetroplach is a more playful name for the anemometer, suggested by
  the author's wife, replacing the Norse god name
- the board and firmware directories, the shared KiCad symbol and
  footprint libraries, the CI workflows, and every in-file reference
  change in one step so the tree never mixes the two names
Parts:
- C1, C2, C3: footprint njordr:C-0805-HandSolder -> vetroplach:C-0805-HandSolder
- C28, C29, R1, R2: footprint njordr:C-0603-HandSolder -> vetroplach:C-0603-HandSolder
- D1: footprint njordr:D-SOD-323-HandSolder -> vetroplach:D-SOD-323-HandSolder
- IC1: footprint njordr:TSSOP-20-4.4x6.5 -> vetroplach:TSSOP-20-4.4x6.5; symbol njordr:DRV8300DPWR -> vetroplach:DRV8300DPWR
- L1: footprint njordr:L-Axial-L7.0-D3.3mm-P10.16 -> vetroplach:L-Axial-L7.0-D3.3mm-P10.16
- R17, R18, R3: footprint njordr:R-0603-HandSolder -> vetroplach:R-0603-HandSolder
- T3, T4: footprint njordr:TestPoint-Pad-1.0x1.0 -> vetroplach:TestPoint-Pad-1.0x1.0
- U2: footprint njordr:SOT-23-6-HandSolder -> vetroplach:SOT-23-6-HandSolder
Other:
- title: NJORDR-BOARD -> VETROPLACH-BOARD
