File: vetroplach-board/power-supply.kicad_sch (KiCad schematic)
At the start: 14 parts, among them T3 TestPoint, T4 TestPoint, T5 TestPoint, T6 TestPoint, U1 MT3608, U2 AMS1117-3.3

Commit message: repo: Rename project from njordr to vetroplach
- vetroplach is a more playful name for the anemometer, suggested by
  the author's wife, replacing the Norse god name
- the board and firmware directories, the shared KiCad symbol and
  footprint libraries, the CI workflows, and every in-file reference
  change in one step so the tree never mixes the two names
Other:
- title: NJORDR-BOARD -> VETROPLACH-BOARD
Changed lines of the file:
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@@
 	(paper "A4")
 	(title_block
-		(title "NJORDR-BOARD")
+		(title "VETROPLACH-BOARD")
 		(date "2025-08-24")
 		(rev "0.1")
@@
 		)
 		(instances
-			(project "njordr-board"
+			(project "vetroplach-board"
 				(path "/837a3018-1957-4824-b018-c0ef83e9cb67/085e2257-4ead-4630-86ba-fd69b8cd726d"
 					(reference "#PWR08")
@@
 		)
 		(instances
-			(project "njordr-board"
+			(project "vetroplach-board"
 				(path "/837a3018-1957-4824-b018-c0ef83e9cb67/085e2257-4ead-4630-86ba-fd69b8cd726d"
 					(reference "R1")
@@
 		)
 		(instances
-			(project "njordr-board"
+			(project "vetroplach-board"
 				(path "/837a3018-1957-4824-b018-c0ef83e9cb67/085e2257-4ead-4630-86ba-fd69b8cd726d"
 					(reference "C2")
@@
 		)
 		(instances
-			(project "njordr-board"
+			(project "vetroplach-board"
 				(path "/837a3018-1957-4824-b018-c0ef83e9cb67/085e2257-4ead-4630-86ba-fd69b8cd726d"
 					(reference "R3")
@@
 		)
 		(instances
-			(project "njordr-board"
+			(project "vetroplach-board"
 				(path "/837a3018-1957-4824-b018-c0ef83e9cb67/085e2257-4ead-4630-86ba-fd69b8cd726d"
 					(reference "C3")
@@
 		)
 		(instances
-			(project "njordr-board"
+			(project "vetroplach-board"
 				(path "/837a3018-1957-4824-b018-c0ef83e9cb67/085e2257-4ead-4630-86ba-fd69b8cd726d"
 					(reference "#PWR02")
@@
 		)
 		(instances
-			(project "njordr-board"
+			(project "vetroplach-board"
 				(path "/837a3018-1957-4824-b018-c0ef83e9cb67/085e2257-4ead-4630-86ba-fd69b8cd726d"
 					(reference "#PWR03")
@@
 		)
 		(instances
-			(project "njordr-board"
+			(project "vetroplach-board"
 				(path "/837a3018-1957-4824-b018-c0ef83e9cb67/085e2257-4ead-4630-86ba-fd69b8cd726d"
 					(reference "#PWR06")
@@
 		)
 		(instances
-			(project "njordr-board"
+			(project "vetroplach-board"
 				(path "/837a3018-1957-4824-b018-c0ef83e9cb67/085e2257-4ead-4630-86ba-fd69b8cd726d"
 					(reference "#FLG02")
@@
 		)
 		(instances
-			(project "njordr-board"
+			(project "vetroplach-board"
 				(path "/837a3018-1957-4824-b018-c0ef83e9cb67/085e2257-4ead-4630-86ba-fd69b8cd726d"
 					(reference "R2")
@@
 		)
 		(instances
-			(project "njordr-board"
+			(project "vetroplach-board"
 				(path "/837a3018-1957-4824-b018-c0ef83e9cb67/085e2257-4ead-4630-86ba-fd69b8cd726d"
 					(reference "#FLG01")
@@
 		)
 		(instances
-			(project "njordr-board"
+			(project "vetroplach-board"
 				(path "/837a3018-1957-4824-b018-c0ef83e9cb67/085e2257-4ead-4630-86ba-fd69b8cd726d"
 					(reference "T3")
@@
 		)
 		(instances
-			(project "njordr-board"
+			(project "vetroplach-board"
 				(path "/837a3018-1957-4824-b018-c0ef83e9cb67/085e2257-4ead-4630-86ba-fd69b8cd726d"
 					(reference "#PWR07")
@@
 		)
 		(instances
-			(project "njordr-board"
+			(project "vetroplach-board"
 				(path "/837a3018-1957-4824-b018-c0ef83e9cb67/085e2257-4ead-4630-86ba-fd69b8cd726d"
 					(reference "U2")
@@
 		)
 		(instances
-			(project "njordr-board"
+			(project "vetroplach-board"
 				(path "/837a3018-1957-4824-b018-c0ef83e9cb67/085e2257-4ead-4630-86ba-fd69b8cd726d"
 					(reference "T4")
@@
 		)
 		(instances
-			(project "njordr-board"
+			(project "vetroplach-board"
 				(path "/837a3018-1957-4824-b018-c0ef83e9cb67/085e2257-4ead-4630-86ba-fd69b8cd726d"
 					(reference "#PWR01")
@@
 		)
 		(instances
-			(project "njordr-board"
+			(project "vetroplach-board"
 				(path "/837a3018-1957-4824-b018-c0ef83e9cb67/085e2257-4ead-4630-86ba-fd69b8cd726d"
 					(reference "T5")
@@
 		)
 		(instances
-			(project "njordr-board"
+			(project "vetroplach-board"
 				(path "/837a3018-1957-4824-b018-c0ef83e9cb67/085e2257-4ead-4630-86ba-fd69b8cd726d"
 					(reference "#PWR04")
@@
 		)
 		(instances
-			(project "njordr-board"
+			(project "vetroplach-board"
 				(path "/837a3018-1957-4824-b018-c0ef83e9cb67/085e2257-4ead-4630-86ba-fd69b8cd726d"
 					(reference "#PWR05")
@@
 		)
 		(instances
-			(project "njordr-board"
+			(project "vetroplach-board"
 				(path "/837a3018-1957-4824-b018-c0ef83e9cb67/085e2257-4ead-4630-86ba-fd69b8cd726d"
 					(reference "T6")
@@
 		)
 		(instances
-			(project "njordr-board"
+			(project "vetroplach-board"
 				(path "/837a3018-1957-4824-b018-c0ef83e9cb67/085e2257-4ead-4630-86ba-fd69b8cd726d"
 					(reference "#PWR09")
@@
 		)
 		(instances
-			(project "njordr-board"
+			(project "vetroplach-board"
 				(path "/837a3018-1957-4824-b018-c0ef83e9cb67/085e2257-4ead-4630-86ba-fd69b8cd726d"
 					(reference "#PWR010")
