File: vetroplach-board/signal-priming.kicad_sch (KiCad schematic)
At the start: 42 parts, among them IC2 GS8054, IC3 TMUX741x, T1 TestPoint, T10 TestPoint, T11 TestPoint, T2 TestPoint, T9 TestPoint, U3 REF3012, U7 LM393

Commit message: repo: Rename project from njordr to vetroplach
- vetroplach is a more playful name for the anemometer, suggested by
  the author's wife, replacing the Norse god name
- the board and firmware directories, the shared KiCad symbol and
  footprint libraries, the CI workflows, and every in-file reference
  change in one step so the tree never mixes the two names
Parts:
- C11, C13, C17, C20, C30, C32, C6, C7, C9: footprint njordr:C-0603-HandSolder -> vetroplach:C-0603-HandSolder
- C18, C21, C31: footprint njordr:C-0805-HandSolder -> vetroplach:C-0805-HandSolder
- D3, D4: footprint njordr:D-SOD-323-HandSolder -> vetroplach:D-SOD-323-HandSolder
- IC2: footprint njordr:TSSOP-14-4.4x5.0 -> vetroplach:TSSOP-14-4.4x5.0; symbol njordr:TL974IPWR -> vetroplach:TL974IPWR
- IC3: footprint njordr:WQFN-16-4.0x4.0 -> vetroplach:WQFN-16-4.0x4.0; symbol njordr:TMUX741x -> vetroplach:TMUX741x
- R10, R11, R12, R13, R14, R15, R16, R19, R20, R21, R22, R23, R24, R25, R26: footprint njordr:R-0603-HandSolder -> vetroplach:R-0603-HandSolder
- T1, T10, T11, T2, T9: footprint njordr:TestPoint-Pad-1.0x1.0 -> vetroplach:TestPoint-Pad-1.0x1.0
- U3: footprint njordr:SOT-23 -> vetroplach:SOT-23
- U7: footprint njordr:SOIC-8-3.9x4.9-P1.27 -> vetroplach:SOIC-8-3.9x4.9-P1.27
