File: vetroplach-board/sonic-channel.kicad_sch (KiCad schematic)
At the start: 26 parts, among them Q101 2N7002, Q102 2N7002, T101 TestPoint, T102 TestPoint, T103 TestPoint, T104 TestPoint, T105 TestPoint, T106 TestPoint, T107 TestPoint

Commit message: repo: Rename project from njordr to vetroplach
- vetroplach is a more playful name for the anemometer, suggested by
  the author's wife, replacing the Norse god name
- the board and firmware directories, the shared KiCad symbol and
  footprint libraries, the CI workflows, and every in-file reference
  change in one step so the tree never mixes the two names
Parts:
- C101, C102, C105, C106, C107, C108: footprint njordr:C-0603-HandSolder -> vetroplach:C-0603-HandSolder
- C103: footprint njordr:C-1206-HandSolder -> vetroplach:C-1206-HandSolder
- C104: footprint njordr:C-0805-HandSolder -> vetroplach:C-0805-HandSolder
- D101, D102: footprint njordr:D-SOD-323-HandSolder -> vetroplach:D-SOD-323-HandSolder
- L101: footprint njordr:L-Axial-L12.0-D5.0-P15.24 -> vetroplach:L-Axial-L12.0-D5.0-P15.24
- Q101, Q102: footprint njordr:SOT-23 -> vetroplach:SOT-23
- R101, R102, R103, R104: footprint njordr:R-0603-HandSolder -> vetroplach:R-0603-HandSolder
- R105: footprint njordr:R-0805-HandSolder -> vetroplach:R-0805-HandSolder
- ST101: footprint njordr:CUSA-TR65-065-2200-TH68 -> vetroplach:CUSA-TR65-065-2200-TH68
- T101, T102, T103, T104, T105, T106, T107: footprint njordr:TestPoint-Pad-1.0x1.0 -> vetroplach:TestPoint-Pad-1.0x1.0
Other:
- title: NJORDR-BOARD -> VETROPLACH-BOARD
