File: vetroplach-board/vetroplach-board.kicad_pcb (KiCad board)
At the start: 4 copper layers, 88 x 80 mm, 132 parts, among them IC1 DRV8300DPWR, IC2 GS8054, IC3 TMUX741x, J1 Conn_01x06, J2 Conn_01x06, J3 Conn_01x06, Q101 2N7002, Q102 2N7002, Q201 2N7002, Q202 2N7002, Q301 2N7002, Q302 2N7002, T1 TestPoint, T10 TestPoint, T101 TestPoint, T102 TestPoint, T103 TestPoint, T104 TestPoint, T105 TestPoint, T106 TestPoint, T107 TestPoint, T11 TestPoint, T2 TestPoint, T201 TestPoint, T202 TestPoint, T203 TestPoint, T204 TestPoint, T205 TestPoint, T206 TestPoint, T207 TestPoint, T3 TestPoint, T301 TestPoint, T302 TestPoint, T303 TestPoint, T304 TestPoint, T305 TestPoint, T306 TestPoint, T307 TestPoint, T4 TestPoint, T9 TestPoint, U2 MT3608, U3 REF3012, U7 LM393

Commit message: repo: Rename project from njordr to vetroplach
- vetroplach is a more playful name for the anemometer, suggested by
  the author's wife, replacing the Norse god name
- the board and firmware directories, the shared KiCad symbol and
  footprint libraries, the CI workflows, and every in-file reference
  change in one step so the tree never mixes the two names
Parts:
- C1, C104, C18, C2, C204, C21, C304, C31: footprint njordr:C-0805-HandSolder -> vetroplach:C-0805-HandSolder
- C101, C102, C105, C106, C107, C108, C11, C13, C17, C20, C201, C202, C205, C206, C207, C208, C28, C29, C30, C301, C302, C305, C306, C307, C308, C32, C6, C7, C9: footprint njordr:C-0603-HandSolder -> vetroplach:C-0603-HandSolder
- C103, C203, C303: footprint njordr:C-1206-HandSolder -> vetroplach:C-1206-HandSolder
- D1, D101, D102, D201, D202, D3, D301, D302, D4: footprint njordr:D-SOD-323-HandSolder -> vetroplach:D-SOD-323-HandSolder
- IC1: footprint njordr:TSSOP-20-4.4x6.5 -> vetroplach:TSSOP-20-4.4x6.5
- IC2: footprint njordr:TSSOP-14-4.4x5.0 -> vetroplach:TSSOP-14-4.4x5.0
- IC3: footprint njordr:WQFN-16-4.0x4.0 -> vetroplach:WQFN-16-4.0x4.0
- J1, J2, J3: footprint njordr:PinHeader-1x06-P2.54mm-Vertical -> vetroplach:PinHeader-1x06-P2.54mm-Vertical
- L1: footprint njordr:L-Axial-L7.0-D3.3mm-P10.16 -> vetroplach:L-Axial-L7.0-D3.3mm-P10.16
- L101, L201, L301: footprint njordr:L-Axial-L12.0-D5.0-P15.24 -> vetroplach:L-Axial-L12.0-D5.0-P15.24
- Q101, Q102, Q201, Q202, Q301, Q302, U3: footprint njordr:SOT-23 -> vetroplach:SOT-23
- R10, R101, R102, R103, R104, R11, R12, R13, R14, R15, R16, R17, R18, R19, R20, R201, R202, R203, R204, R21, R22, R23, R24, R25, R26, R3, R301, R302, R303, R304: footprint njordr:R-0603-HandSolder -> vetroplach:R-0603-HandSolder
- R105, R205, R305: footprint njordr:R-0805-HandSolder -> vetroplach:R-0805-HandSolder
- ST101, ST201, ST301: footprint njordr:CUSA-TR65-065-2200-TH68 -> vetroplach:CUSA-TR65-065-2200-TH68
- T1, T10, T101, T102, T103, T104, T105, T106, T107, T11, T2, T201, T202, T203, T204, T205, T206, T207, T3, T301, T302, T303, T304, T305, T306, T307, T4, T9: footprint njordr:TestPoint-Pad-1.0x1.0 -> vetroplach:TestPoint-Pad-1.0x1.0
- U2: footprint njordr:SOT-23-6-HandSolder -> vetroplach:SOT-23-6-HandSolder
- U7: footprint njordr:SOIC-8-3.9x4.9-P1.27 -> vetroplach:SOIC-8-3.9x4.9-P1.27
Other:
- board text added: "VETROPLACH-BOARD 251025 JKR"
- board text removed: "NJORDR-BOARD 251025 JKR"
