File: vetroplach-board/vetroplach-board.kicad_sch (KiCad schematic)
At the start: 3 parts, among them J1 Conn_01x06, J2 Conn_01x06, J3 Conn_01x06

Commit message: repo: Rename project from njordr to vetroplach
- vetroplach is a more playful name for the anemometer, suggested by
  the author's wife, replacing the Norse god name
- the board and firmware directories, the shared KiCad symbol and
  footprint libraries, the CI workflows, and every in-file reference
  change in one step so the tree never mixes the two names
Parts:
- J1, J2, J3: footprint njordr:PinHeader-1x06-P2.54mm-Vertical -> vetroplach:PinHeader-1x06-P2.54mm-Vertical
Other:
- title: NJORDR-BOARD -> VETROPLACH-BOARD
Changed lines of the file:
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@@
 	(paper "A4")
 	(title_block
-		(title "NJORDR-BOARD")
+		(title "VETROPLACH-BOARD")
 		(date "2025-08-24")
 		(rev "0.1")
@@
 		)
 		(instances
-			(project "njordr-board"
+			(project "vetroplach-board"
 				(path "/837a3018-1957-4824-b018-c0ef83e9cb67"
 					(reference "#PWR051")
@@
 		)
 		(instances
-			(project "njordr-board"
+			(project "vetroplach-board"
 				(path "/837a3018-1957-4824-b018-c0ef83e9cb67"
 					(reference "#PWR046")
@@
 			)
 		)
-		(property "Footprint" "njordr:PinHeader-1x06-P2.54mm-Vertical"
+		(property "Footprint" "vetroplach:PinHeader-1x06-P2.54mm-Vertical"
 			(at 60.96 91.44 0)
 			(effects
@@
 		)
 		(instances
-			(project "njordr-board"
+			(project "vetroplach-board"
 				(path "/837a3018-1957-4824-b018-c0ef83e9cb67"
 					(reference "J2")
@@
 		)
 		(instances
-			(project "njordr-board"
+			(project "vetroplach-board"
 				(path "/837a3018-1957-4824-b018-c0ef83e9cb67"
 					(reference "#PWR048")
@@
 		)
 		(instances
-			(project "njordr-board"
+			(project "vetroplach-board"
 				(path "/837a3018-1957-4824-b018-c0ef83e9cb67"
 					(reference "#PWR049")
@@
 			)
 		)
-		(property "Footprint" "njordr:PinHeader-1x06-P2.54mm-Vertical"
+		(property "Footprint" "vetroplach:PinHeader-1x06-P2.54mm-Vertical"
 			(at 60.96 116.84 0)
 			(effects
@@
 		)
 		(instances
-			(project "njordr-board"
+			(project "vetroplach-board"
 				(path "/837a3018-1957-4824-b018-c0ef83e9cb67"
 					(reference "J3")
@@
 			)
 		)
-		(property "Footprint" "njordr:PinHeader-1x06-P2.54mm-Vertical"
+		(property "Footprint" "vetroplach:PinHeader-1x06-P2.54mm-Vertical"
 			(at 60.96 66.04 0)
 			(effects
@@
 		)
 		(instances
-			(project "njordr-board"
+			(project "vetroplach-board"
 				(path "/837a3018-1957-4824-b018-c0ef83e9cb67"
 					(reference "#PWR050")
@@
 		)
 		(instances
-			(project "njordr-board"
+			(project "vetroplach-board"
 				(path "/837a3018-1957-4824-b018-c0ef83e9cb67"
 					(reference "#PWR047")
@@
 		)
 		(instances
-			(project "njordr-board"
+			(project "vetroplach-board"
 				(path "/837a3018-1957-4824-b018-c0ef83e9cb67"
 					(page "4")
@@
 		)
 		(instances
-			(project "njordr-board"
+			(project "vetroplach-board"
 				(path "/837a3018-1957-4824-b018-c0ef83e9cb67"
 					(page "5")
@@
 		)
 		(instances
-			(project "njordr-board"
+			(project "vetroplach-board"
 				(path "/837a3018-1957-4824-b018-c0ef83e9cb67"
 					(page "7")
@@
 		)
 		(instances
-			(project "njordr-board"
+			(project "vetroplach-board"
 				(path "/837a3018-1957-4824-b018-c0ef83e9cb67"
 					(page "6")
@@
 		)
 		(instances
-			(project "njordr-board"
+			(project "vetroplach-board"
 				(path "/837a3018-1957-4824-b018-c0ef83e9cb67"
 					(page "3")
@@
 		)
 		(instances
-			(project "njordr-board"
+			(project "vetroplach-board"
 				(path "/837a3018-1957-4824-b018-c0ef83e9cb67"
 					(page "2")
